File: hardware/main-board/main-board.kicad_pcb (KiCad board)
At the start: 4 copper layers, 50 x 50 mm, 57 parts, among them J1 Conn_01x04_Socket, J2 Conn_01x04_Socket, J5 USB_C_Receptacle_USB2.0_16P, J6 Conn_01x02_MountingPin, Q1 DMG3415U-7, SW1 SW_SPDT, SW5 SW_Push, SW7 SW_Push, SW8 SW_Push, U1 ESP32-C6-MINI-1/U, U2 USBLC6-2SC6, U3 AP2112K-3.3, U4 TP4056-42-ESOP8

Commit message: Added overvoltage protection to schematic
Layout Needs to be rerouted
Parts:
- added C13: 10u, Capacitor_SMD:C_1206_3216Metric_Pad1.33x1.80mm_HandSolder, F.Cu at (154.0, 144.0)
- added C14: 100u, Capacitor_SMD:C_1210_3225Metric_Pad1.33x2.70mm_HandSolder, F.Cu at (154.0, 147.8)
- added C16: 100n, Capacitor_SMD:C_0805_2012Metric_Pad1.18x1.45mm_HandSolder, F.Cu at (159.4, 143.8)
- added R23: 10k, Resistor_SMD:R_0805_2012Metric_Pad1.20x1.40mm_HandSolder, F.Cu at (159.3, 151.9)
- added U5: AP22815AWT-7, Package_TO_SOT_SMD:SOT-23-5_HandSoldering, F.Cu at (158.6, 133.6)
- D12: value SS14 -> MBR120LSFT1G; footprint Diode_SMD:D_SMA_Handsoldering -> Diode_SMD:D_SOD-123F
- Q1: value DMG3415U-7 -> DMG2305UX
Connections:
- net /VBUS renamed /VBUS_PROTECTION_IN
- F1 pad 2: +5V -> Net-(U5-EN)
Other:
- board text added: "Needs to find a place and reroute power"

Commit message: After deciding we wont include OVP in this design, so i removed it from active schematic and check if everything is alright in pcb
Parts:
- removed C13: 10u, Capacitor_SMD:C_1206_3216Metric_Pad1.33x1.80mm_HandSolder
- removed C14: 100u, Capacitor_SMD:C_1210_3225Metric_Pad1.33x2.70mm_HandSolder
- removed C16: 100n, Capacitor_SMD:C_0805_2012Metric_Pad1.18x1.45mm_HandSolder
- removed R23: 10k, Resistor_SMD:R_0805_2012Metric_Pad1.20x1.40mm_HandSolder
- removed U5: AP22815AWT-7, Package_TO_SOT_SMD:SOT-23-5_HandSoldering
Connections:
- net /VBUS_PROTECTION_IN renamed Net-(D8-A2)
- F1 pad 2: Net-(U5-EN) -> +5V
Other:
- board text removed: "Needs to find a place and reroute power"
